File: hardware/usbasp.brd (EAGLE design)
At the start: 34.9 x 16.5 mm, 25 parts, among them IC1 ATMEGA8-16A, Q2 12Mhz, X1 USB-A-H

Commit message: hardware: coscmetic fixes
Parts:
- C5: value 0.1u -> 100n
- D1, D2: value (none) -> 3V6
Connections:
- net N$1 renamed XTAL1
- net N$10 renamed SLOWSCK
- net N$2 renamed XTAL2
Changed lines of the file:
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@@
 <element name="R4" library="rcl" package="M0805" value="68" x="7.62" y="13.335" rot="R270"/>
 <element name="C4" library="rcl" package="SMC_A" value="10u" x="1.016" y="8.89" rot="MR90"/>
-<element name="C5" library="rcl" package="C0805" value="0.1u" x="15.24" y="9.525" rot="MR90"/>
+<element name="C5" library="rcl" package="C0805" value="100n" x="15.24" y="9.525" rot="MR90"/>
 <element name="WRITE" library="led" package="CHIP-LED0805" value="" x="32.385" y="2.54" rot="R90"/>
 <element name="ACTIVE" library="led" package="CHIP-LED0805" value="" x="32.385" y="13.97" rot="R90"/>
@@
 <element name="SELF" library="pinhead" package="1X02" value="" x="25.4" y="3.175"/>
 <element name="IC1" library="avr" package="TQFP32-08" value="ATMEGA8-16A" x="16.51" y="9.525"/>
-<element name="D2" library="sparkfun" package="SMA-DIODE" value="" x="7.62" y="4.445" rot="MR90"/>
-<element name="D1" library="sparkfun" package="SMA-DIODE" value="" x="7.62" y="12.065" rot="MR270"/>
+<element name="D2" library="sparkfun" package="SMA-DIODE" value="3V6" x="7.62" y="4.445" rot="MR90"/>
+<element name="D1" library="sparkfun" package="SMA-DIODE" value="3V6" x="7.62" y="12.065" rot="MR270"/>
 <element name="X1" library="sparkfun" package="USB-A-H" value="USB-A-H" x="2.54" y="8.255"/>
 <element name="ISP1" library="balto" package="2X03_BORDER" value="" x="33.02" y="8.255" rot="R270"/>
@@
 </elements>
 <signals>
-<signal name="N$1">
+<signal name="XTAL1">
 <contactref element="Q2" pad="2"/>
 <contactref element="C1" pad="2"/>
@@
 <via x="11.176" y="5.6896" extent="1-16" drill="0.508"/>
 </signal>
-<signal name="N$2">
+<signal name="XTAL2">
 <contactref element="C3" pad="2"/>
 <contactref element="Q2" pad="1"/>
@@
 <via x="33.3248" y="15.4432" extent="1-16" drill="0.508"/>
 </signal>
-<signal name="N$10">
+<signal name="SLOWSCK">
 <contactref element="SLOWSCK" pad="1"/>
 <contactref element="IC1" pad="25"/>
