File: hardware/usbasp-rev2.brd (EAGLE design)
At the start: 29.7 x 15.4 mm, 29 parts, among them IC1 ATMEGA8-16A, U1 MIC2551, X1 USB-A-H, Y1 12MHz

Commit message: hw: rev2: fix ldo part number
Parts:
- U1: value MIC2551 -> MIC5301
Changed lines of the file:
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@@
 </element>
 <element name="R7" library="rcl" package="R0805" value="10" x="23.7744" y="2.032"/>
-<element name="U1" library="SparkFun-PowerIC" package="SOT23-5" value="MIC2551" x="7.7216" y="2.032" rot="R270"/>
+<element name="U1" library="SparkFun-PowerIC" package="SOT23-5" value="MIC5301" x="7.7216" y="2.032" rot="R270"/>
 <element name="C6" library="rcl" package="C0603" value=".1u" x="11.3792" y="1.016"/>
 <element name="C7" library="rcl" package="C0603" value=".1u" x="7.7216" y="4.064"/>
