File: hardware/usbasp-rev2.brd (EAGLE design)
At the start: 29.7 x 15.4 mm, 29 parts, among them IC1 ATMEGA8-16A, U1 MIC5301, X1 USB-A-H, Y1 12MHz

Commit message: hw: update part values
Parts:
- ACTIVE: value (none) -> RED
- R5, R6: value 1k -> 470
- R7: value 10 -> 1
- R8: value 1k -> 4k7
- WRITE: value (none) -> GREEN
Changed lines of the file:
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@@
 <element name="R4" library="rcl" package="R0603" value="68" x="7.5184" y="9.3472" rot="R180"/>
 <element name="C5" library="rcl" package="C0603" value=".1u" x="14.6304" y="7.9248" rot="MR180"/>
-<element name="WRITE" library="led" package="CHIP-LED0805" value="" x="27.432" y="3.048" rot="R90"/>
-<element name="ACTIVE" library="led" package="CHIP-LED0805" value="" x="27.432" y="12.3952" rot="R90"/>
-<element name="R5" library="rcl" package="R0603" value="1k" x="27.432" y="3.048" rot="MR180"/>
-<element name="R6" library="rcl" package="R0603" value="1k" x="27.432" y="12.3952" rot="MR180"/>
+<element name="WRITE" library="led" package="CHIP-LED0805" value="GREEN" x="27.432" y="3.048" rot="R90"/>
+<element name="ACTIVE" library="led" package="CHIP-LED0805" value="RED" x="27.432" y="12.3952" rot="R90"/>
+<element name="R5" library="rcl" package="R0603" value="470" x="27.432" y="3.048" rot="MR180"/>
+<element name="R6" library="rcl" package="R0603" value="470" x="27.432" y="12.3952" rot="MR180"/>
 <element name="IC1" library="avr" package="TQFP32-08" value="ATMEGA8-16A" x="14.8336" y="7.7216"/>
 <element name="D2" library="sparkfun" package="SMA-DIODE" value="3V6" x="7.5184" y="4.6736" rot="MR90"/>
@@
 <attribute name="TP_SIGNAL_NAME" value="" x="37.592" y="-25.7556" size="1.778" layer="27" display="off"/>
 </element>
-<element name="R7" library="rcl" package="R0805" value="10" x="23.7744" y="2.032"/>
+<element name="R7" library="rcl" package="R0805" value="1" x="23.7744" y="2.032"/>
 <element name="U1" library="SparkFun-PowerIC" package="SOT23-5" value="MIC5301" x="7.7216" y="2.032" rot="R270"/>
 <element name="C6" library="rcl" package="C0603" value=".1u" x="11.3792" y="1.016"/>
@@
 <attribute name="OC_FARNELL" value="unknown" x="4.1148" y="28.0416" size="1.778" layer="27" rot="R180" display="off"/>
 </element>
-<element name="R8" library="rcl" package="R0603" value="1k" x="21.7424" y="9.144" rot="MR315"/>
+<element name="R8" library="rcl" package="R0603" value="4k7" x="21.7424" y="9.144" rot="MR315"/>
 <element name="R9" library="rcl" package="R0603" value="1k" x="20.7264" y="6.9088" rot="MR225"/>
 </elements>
@@
 </signal>
 </signals>
-<errors>
-</errors>
 </board>
 </drawing>
